File: schematics/sketchingpad/sketchingpad.kicad_pcb (KiCad board)
At the start: 2 copper layers, 120 x 90 mm, 57 parts, among them J1 Conn_01x07, J2 Conn_01x07, SW1 Capacitive_Button, SW10 Capacitive_Button, SW11 Capacitive_Button, SW12 Capacitive_Button, SW13 Capacitive_Button, SW14 Capacitive_Button, SW15 Capacitive_Button, SW16 Capacitive_Button, SW17 Capacitive_Button, SW18 Capacitive_Button, SW19 Capacitive_Button, SW2 Capacitive_Button, SW20 Capacitive_Button, SW3 Capacitive_Button, SW4 Capacitive_Button, SW5 Capacitive_Button, SW6 Capacitive_Button, SW7 Capacitive_Button, SW8 Capacitive_Button, SW9 Capacitive_Button, U1 TS20, U2 IS31FL3731-SA, U5 XIAO-ESP32-S3-SMD

Commit message: some pcb layout for touch
Parts:
- removed U5: XIAO-ESP32-S3-SMD, Seeed Studio XIAO Series Library:XIAO-ESP32C6-SMD
- SW10, SW12, SW2, SW4, SW6, SW8: footprint todbot_stuff:Pad-Captouch-0.5in-backlitD -> todbot_stuff:Pad-Captouch-0.5in-backlitB
- moved SW1 99.0 mm to (87.0, 113.0)
- moved SW7 81.7 mm to (104.0, 117.0)
- moved SW11 70.6 mm to (99.0, 132.0)
- moved LED19 67.2 mm to (185.2, 140.8)
- moved LED6 66.9 mm to (185.0, 107.5)
- moved LED20 60.1 mm to (184.0, 81.5)
- moved LED14 56.5 mm to (173.0, 126.2)
- moved LED22 52.7 mm to (172.5, 83.0)
- moved LED25 50.3 mm to (172.5, 78.0)
- moved LED5 49.5 mm to (166.5, 94.5)
- moved SW20 49.0 mm to (184.0, 87.0)
- moved LED18 48.1 mm to (161.0, 143.5)
- moved LED23 47.5 mm to (173.0, 89.5)
- moved LED15 46.9 mm to (87.0, 140.5)
- moved LED24 45.2 mm to (168.0, 83.5)
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Connections:
- U1 pad 1: /TOUCH5 -> /TOUCH4
- U1 pad 11: /TOUCH13 -> /TOUCH19
- U1 pad 12: /TOUCH14 -> /TOUCH18
- U1 pad 13: /TOUCH15 -> /TOUCH17
- U1 pad 15: /TOUCH17 -> /TOUCH15
- U1 pad 16: unconnected-(U1-CS18-Pad16) -> /TOUCH11
- U1 pad 17: unconnected-(U1-CS19-Pad17) -> /TOUCH1
- U1 pad 18: unconnected-(U1-CS20-Pad18) -> /TOUCH7
- U1 pad 2: /TOUCH6 -> /TOUCH9
- U1 pad 25: /TOUCH1 -> /TOUCH12
- U1 pad 27: /TOUCH3 -> /TOUCH8
- U1 pad 28: /TOUCH4 -> /TOUCH3
- U1 pad 3: /TOUCH7 -> /TOUCH5
- U1 pad 5: /TOUCH8 -> /TOUCH20
- U1 pad 6: /TOUCH9 -> /TOUCH10
- U1 pad 7: /TOUCH10 -> /TOUCH6
- U1 pad 8: /TOUCH11 -> /TOUCH13
- U1 pad 9: /TOUCH12 -> /TOUCH14
Routing:
- net /TOUCH20: track 0.00 -> 74.6 mm, vias 0 -> 1
- net /TOUCH1: track 0.00 -> 62.2 mm, vias 0 -> 1
- net /TOUCH6: track 0.00 -> 61.0 mm, vias 0 -> 1
- net /TOUCH19: track 0.00 -> 59.2 mm, vias 0 -> 1
- net /TOUCH15: track 0.00 -> 57.9 mm, vias 0 -> 1
- net /TOUCH2: track 0.00 -> 49.9 mm, vias 0 -> 1
- net /TOUCH16: track 0.00 -> 48.6 mm, vias 0 -> 1
- net /TOUCH5: track 0.00 -> 47.5 mm, vias 0 -> 1
- net /TOUCH7: track 0.00 -> 45.0 mm, vias 0 -> 1
- net /TOUCH14: track 0.00 -> 44.4 mm, vias 0 -> 1
- net /TOUCH11: track 0.00 -> 42.7 mm, vias 0 -> 1
- net /TOUCH10: track 0.00 -> 42.2 mm, vias 0 -> 1
- net /TOUCH18: track 0.00 -> 40.4 mm, vias 0 -> 1
- net /TOUCH3: track 0.00 -> 39.6 mm, vias 0 -> 1
- net /TOUCH4: track 0.00 -> 39.1 mm, vias 0 -> 1
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- added copper zone on In1.Cu, net GND
- added copper zone on In2.Cu, net GND
Other:
- copper layers 2 -> 4

Commit message: some pcb layout for touch
Routing:
- net /CA8: track 0.00 -> 35.0 mm, vias 0 -> 2
- net /CA5: track 0.00 -> 34.2 mm, vias 0 -> 3
- net /SDA: track 0.00 -> 31.8 mm, vias 0 -> 2
- net /SCL: track 0.00 -> 31.1 mm, vias 0 -> 2
- net /CA6: track 0.00 -> 16.9 mm, vias 0 -> 2
- net GND: track 0.00 -> 5.36 mm, vias 0 -> 3
- net /TOUCH2: track 49.9 -> 46.3 mm

Commit message: sketchingpad_proto1: chickening out with sk6812side instead of charlieplex RGB
Parts:
- SW14, SW16, SW18, SW20: footprint todbot_stuff:Pad-Captouch-0.5in-backlitD -> todbot_stuff:Pad-Captouch-0.5in-backlitB
- moved R16 34.4 mm to (129.8, 136.8), turned to 90 degrees
- moved C3 22.2 mm to (136.0, 128.2)
- moved LED23 12.7 mm to (170.5, 77.0)
- moved LED24 11.9 mm to (178.0, 77.0)
- moved LED25 11.5 mm to (184.0, 77.0)
- moved R18 5.13 mm to (88.6, 94.8)
- moved R17 4.88 mm to (88.6, 96.8)
- moved LED21 3.00 mm to (170.5, 89.0)
- moved LED18 2.06 mm to (163.0, 143.0)
- moved LED22 2.00 mm to (170.5, 83.0)
- moved LED16 1.73 mm to (109.2, 143.2)
- moved LED12 0.86 mm to (120.0, 127.2)
- moved LED19 0.78 mm to (185.2, 140.0)
- moved LED5 0.71 mm to (166.0, 94.0)
- moved LED1 0.70 mm to (87.0, 107.0)
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Connections:
- net /SCL renamed /Root/SCL
- net /SDA renamed /Root/SDA
- net /TOUCH1 renamed /Root/TOUCH1
- net /TOUCH10 renamed /Root/TOUCH10
- net /TOUCH11 renamed /Root/TOUCH11
- net /TOUCH12 renamed /Root/TOUCH12
- net /TOUCH13 renamed /Root/TOUCH13
- net /TOUCH14 renamed /Root/TOUCH14
- net /TOUCH15 renamed /Root/TOUCH15
- net /TOUCH16 renamed /Root/TOUCH16
- net /TOUCH17 renamed /Root/TOUCH17
- net /TOUCH18 renamed /Root/TOUCH18
- net /TOUCH19 renamed /Root/TOUCH19
- net /TOUCH2 renamed /Root/TOUCH2
- net /TOUCH20 renamed /Root/TOUCH20
- net /TOUCH3 renamed /Root/TOUCH3
- net /TOUCH4 renamed /Root/TOUCH4
- net /TOUCH5 renamed /Root/TOUCH5
- net /TOUCH6 renamed /Root/TOUCH6
- net /TOUCH7 renamed /Root/TOUCH7
- net /TOUCH8 renamed /Root/TOUCH8
- net /TOUCH9 renamed /Root/TOUCH9
- LED1 pad 1: /CA4 -> /LEDs/CA4
- LED1 pad 2: /CA3 -> /LEDs/CA3
- LED1 pad 3: /CA1 -> /LEDs/CA1
- LED1 pad 4: /CA9 -> /LEDs/CA9
- LED10 pad 1: /CA7 -> /LEDs/CA7
- LED10 pad 2: /CA6 -> /LEDs/CA6
- LED10 pad 3: /CA3 -> /LEDs/CA3
- LED10 pad 4: /CA8 -> /LEDs/CA8
- LED11 pad 1: /CA7 -> /LEDs/CA7
- LED11 pad 2: /CA6 -> /LEDs/CA6
- LED11 pad 3: /CA4 -> /LEDs/CA4
- LED11 pad 4: /CA8 -> /LEDs/CA8
- LED12 pad 1: /CA7 -> /LEDs/CA7
- LED12 pad 2: /CA6 -> /LEDs/CA6
- LED12 pad 3: /CA5 -> /LEDs/CA5
- LED12 pad 4: /CA8 -> /LEDs/CA8
- LED13 pad 1: /CA7 -> /LEDs/CA7
- LED13 pad 2: /CA5 -> /LEDs/CA5
- LED13 pad 3: /CA6 -> /LEDs/CA6
- LED13 pad 4: /CA8 -> /LEDs/CA8
- LED14 pad 1: /CA6 -> /LEDs/CA6
- LED14 pad 2: /CA5 -> /LEDs/CA5
- LED14 pad 3: /CA7 -> /LEDs/CA7
- LED14 pad 4: /CA8 -> /LEDs/CA8
- LED15 pad 1: /CB4 -> /LEDs/CB4
- LED15 pad 2: /CB3 -> /LEDs/CB3
- LED15 pad 3: /CB9 -> /LEDs/CB9
- LED15 pad 4: /CB8 -> /LEDs/CB8
- LED16 pad 1: /CB4 -> /LEDs/CB4
- LED16 pad 2: /CB3 -> /LEDs/CB3
- LED16 pad 3: /CB2 -> /LEDs/CB2
- LED16 pad 4: /CB8 -> /LEDs/CB8
- LED17 pad 1: /CB4 -> /LEDs/CB4
- LED17 pad 2: /CB2 -> /LEDs/CB2
- LED17 pad 3: /CB3 -> /LEDs/CB3
- LED17 pad 4: /CB8 -> /LEDs/CB8
- LED18 pad 1: /CB3 -> /LEDs/CB3
- LED18 pad 2: /CB2 -> /LEDs/CB2
- LED18 pad 3: /CB4 -> /LEDs/CB4
- LED18 pad 4: /CB8 -> /LEDs/CB8
- LED19 pad 1: /CB3 -> /LEDs/CB3
- LED19 pad 2: /CB2 -> /LEDs/CB2
- LED19 pad 3: /CB5 -> /LEDs/CB5
- LED19 pad 4: /CB8 -> /LEDs/CB8
- LED2 pad 1: /CA4 -> /LEDs/CA4
- LED2 pad 2: /CA3 -> /LEDs/CA3
- LED2 pad 3: /CA2 -> /LEDs/CA2
- LED2 pad 4: /CA9 -> /LEDs/CA9
- LED20 pad 1: /CB3 -> /LEDs/CB3
- LED20 pad 2: /CB2 -> /LEDs/CB2
- LED20 pad 3: /CB6 -> /LEDs/CB6
- LED20 pad 4: /CB8 -> /LEDs/CB8
- LED21 pad 1: /CB3 -> /LEDs/CB3
- LED21 pad 2: /CB2 -> /LEDs/CB2
- LED21 pad 3: /CB7 -> /LEDs/CB7
- LED21 pad 4: /CB8 -> /LEDs/CB8
- LED22 pad 1: /CB7 -> /LEDs/CB7
- LED22 pad 2: /CB6 -> /LEDs/CB6
- LED22 pad 3: /CB9 -> /LEDs/CB9
- LED22 pad 4: /CB1 -> /LEDs/CB1
- LED23 pad 1: /CB7 -> /LEDs/CB7
- LED23 pad 2: /CB6 -> /LEDs/CB6
- LED23 pad 3: /CB2 -> /LEDs/CB2
- LED23 pad 4: /CB1 -> /LEDs/CB1
- LED24 pad 1: /CB7 -> /LEDs/CB7
- LED24 pad 2: /CB6 -> /LEDs/CB6
- LED24 pad 3: /CB3 -> /LEDs/CB3
- LED24 pad 4: /CB1 -> /LEDs/CB1
- LED25 pad 1: /CB7 -> /LEDs/CB7
- LED25 pad 2: /CB6 -> /LEDs/CB6
- LED25 pad 3: /CB4 -> /LEDs/CB4
- LED25 pad 4: /CB1 -> /LEDs/CB1
- LED3 pad 1: /CA4 -> /LEDs/CA4
- LED3 pad 2: /CA2 -> /LEDs/CA2
- LED3 pad 3: /CA3 -> /LEDs/CA3
- LED3 pad 4: /CA9 -> /LEDs/CA9
- LED4 pad 1: /CA3 -> /LEDs/CA3
- LED4 pad 2: /CA2 -> /LEDs/CA2
- LED4 pad 3: /CA4 -> /LEDs/CA4
- LED4 pad 4: /CA9 -> /LEDs/CA9
- LED5 pad 1: /CA3 -> /LEDs/CA3
- LED5 pad 2: /CA2 -> /LEDs/CA2
- LED5 pad 3: /CA5 -> /LEDs/CA5
- LED5 pad 4: /CA9 -> /LEDs/CA9
- LED6 pad 1: /CA3 -> /LEDs/CA3
- LED6 pad 2: /CA2 -> /LEDs/CA2
- LED6 pad 3: /CA6 -> /LEDs/CA6
- LED6 pad 4: /CA9 -> /LEDs/CA9
- LED7 pad 1: /CA3 -> /LEDs/CA3
- LED7 pad 2: /CA2 -> /LEDs/CA2
- LED7 pad 3: /CA7 -> /LEDs/CA7
- LED7 pad 4: /CA9 -> /LEDs/CA9
- LED8 pad 1: /CA7 -> /LEDs/CA7
- LED8 pad 2: /CA6 -> /LEDs/CA6
- LED8 pad 3: /CA1 -> /LEDs/CA1
- LED8 pad 4: /CA8 -> /LEDs/CA8
- LED9 pad 1: /CA7 -> /LEDs/CA7
- LED9 pad 2: /CA6 -> /LEDs/CA6
- LED9 pad 3: /CA2 -> /LEDs/CA2
- LED9 pad 4: /CA8 -> /LEDs/CA8
- U2 pad 1: /CA9 -> /Root/CA9
- U2 pad 10: /CB4 -> /Root/CB4
- U2 pad 11: /CB5 -> /Root/CB5
- U2 pad 12: /CB6 -> /Root/CB6
- U2 pad 13: /CB7 -> /Root/CB7
- U2 pad 14: /CB8 -> /Root/CB8
- U2 pad 15: /CB9 -> /Root/CB9
- U2 pad 21: /CA1 -> /Root/CA1
- U2 pad 22: /CA2 -> /Root/CA2
- U2 pad 23: /CA3 -> /Root/CA3
- U2 pad 24: /CA4 -> /Root/CA4
- U2 pad 25: /CA5 -> /Root/CA5
- U2 pad 26: /CA6 -> /Root/CA6
- U2 pad 27: /CA7 -> /Root/CA7
- U2 pad 28: /CA8 -> /Root/CA8
- U2 pad 7: /CB1 -> /Root/CB1
- U2 pad 8: /CB2 -> /Root/CB2
- U2 pad 9: /CB3 -> /Root/CB3
Routing:
- net /Root/SDA: track 31.8 -> 71.3 mm, vias 2 -> 3
- net /CA8: track 35.0 -> 0.00 mm, vias 2 -> 0
- net /CA5: track 34.2 -> 0.00 mm, vias 3 -> 0
- net /Root/SCL: track 31.1 -> 60.1 mm, vias 2 -> 3
- net /CA6: track 16.9 -> 0.00 mm, vias 2 -> 0
- net +3.3V: track 0.00 -> 14.6 mm
- net GND: track 5.36 -> 14.4 mm, vias 3 -> 5
- net /Root/TOUCH1: track 62.2 -> 67.6 mm
- net Net-(U1-INT): track 0.00 -> 3.54 mm
- net /Root/TOUCH15: track 57.9 -> 60.6 mm
- net /Root/TOUCH17: track 33.1 -> 35.3 mm
- net /Root/TOUCH18: track 40.4 -> 39.2 mm
- net /Root/TOUCH14: track 44.4 -> 43.2 mm
- net /Root/TOUCH11: track 42.7 -> 43.7 mm
- net /Root/TOUCH16: track 48.6 -> 49.3 mm
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