File: schematics/sketchingpad/sketchingpad.kicad_sch (KiCad schematic)
At the start: 32 parts, among them J1 Conn_01x07, J2 Conn_01x07, SW1 Capacitive_Button, SW10 Capacitive_Button, SW11 Capacitive_Button, SW12 Capacitive_Button, SW13 Capacitive_Button, SW14 Capacitive_Button, SW15 Capacitive_Button, SW16 Capacitive_Button, SW17 Capacitive_Button, SW18 Capacitive_Button, SW19 Capacitive_Button, SW2 Capacitive_Button, SW20 Capacitive_Button, SW3 Capacitive_Button, SW4 Capacitive_Button, SW5 Capacitive_Button, SW6 Capacitive_Button, SW7 Capacitive_Button, SW8 Capacitive_Button, SW9 Capacitive_Button, U1 TS20, U2 IS31FL3731-SA, U5 XIAO-ESP32-S3-SMD

Commit message: some pcb layout for touch
Parts:
- removed U5: XIAO-ESP32-S3-SMD, Seeed Studio XIAO Series Library:XIAO-ESP32C6-SMD, symbol Seeed_Studio_XIAO_Series:XIAO-ESP32-C6-SMD
- SW10, SW12, SW2, SW4, SW6, SW8: footprint todbot_stuff:Pad-Captouch-0.5in-backlitD -> todbot_stuff:Pad-Captouch-0.5in-backlitB
Connections:
- net TOUCH1: now also U1.17 (CS19); no longer U1.25 (CS1)
- net TOUCH10: now also U1.6 (CS9); no longer U1.7 (CS10)
- net TOUCH11: now also U1.16 (CS18); no longer U1.8 (CS11)
- net TOUCH12: now also U1.25 (CS1); no longer U1.9 (CS12)
- net TOUCH13: now also U1.8 (CS11); no longer U1.11 (CS13)
- net TOUCH14: now also U1.9 (CS12); no longer U1.12 (CS14)
- net TOUCH15: now also U1.15 (CS17); no longer U1.13 (CS15)
- net TOUCH17: now also U1.13 (CS15); no longer U1.15 (CS17)
- net TOUCH18: now also U1.12 (CS14)
- net TOUCH19: now also U1.11 (CS13)
- net TOUCH20: now also U1.3 (CS7)
- net TOUCH3: now also U1.28 (CS4); no longer U1.27 (CS3)
- net TOUCH4: now also U1.1 (CS5); no longer U1.28 (CS4)
- net TOUCH5: now also U1.5 (CS8); no longer U1.1 (CS5)
- net TOUCH6: now also U1.7 (CS10); no longer U1.2 (CS6)
- net TOUCH7: now also U1.18 (CS20); no longer U1.3 (CS7)
- net TOUCH8: now also U1.27 (CS3); no longer U1.5 (CS8)
- net TOUCH9: now also U1.2 (CS6); no longer U1.6 (CS9)
- no-connect marks 3 -> 0

Commit message: some pcb layout for touch
Connections:
- net TOUCH20: now also U1.5 (CS8); no longer U1.3 (CS7)
- net TOUCH5: now also U1.3 (CS7); no longer U1.5 (CS8)
Changed lines of the file:
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@@
 		)
 	)
-	(label "TOUCH5"
+	(label "TOUCH20"
 		(at 208.28 67.31 0)
 		(effects
@@
 		)
 	)
-	(label "TOUCH20"
+	(label "TOUCH5"
 		(at 208.28 64.77 0)
 		(effects

Commit message: sketchingpad_proto1: chickening out with sk6812side instead of charlieplex RGB
Parts:
- SW14, SW16, SW18, SW20: footprint todbot_stuff:Pad-Captouch-0.5in-backlitD -> todbot_stuff:Pad-Captouch-0.5in-backlitB
Changed lines of the file:
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@@
 			)
 		)
-		(property "Footprint" "todbot_stuff:Pad-Captouch-0.5in-backlitD"
+		(property "Footprint" "todbot_stuff:Pad-Captouch-0.5in-backlitB"
 			(at 246.38 121.92 0)
 			(hide yes)
@@
 			)
 		)
-		(property "Footprint" "todbot_stuff:Pad-Captouch-0.5in-backlitD"
+		(property "Footprint" "todbot_stuff:Pad-Captouch-0.5in-backlitB"
 			(at 205.74 120.65 0)
 			(hide yes)
@@
 			)
 		)
-		(property "Footprint" "todbot_stuff:Pad-Captouch-0.5in-backlitD"
+		(property "Footprint" "todbot_stuff:Pad-Captouch-0.5in-backlitB"
 			(at 246.38 135.89 0)
 			(hide yes)
@@
 			)
 		)
-		(property "Footprint" "todbot_stuff:Pad-Captouch-0.5in-backlitD"
+		(property "Footprint" "todbot_stuff:Pad-Captouch-0.5in-backlitB"
 			(at 205.74 134.62 0)
 			(hide yes)
