File: schematics/sketchingpad_proto1/leds.kicad_sch (KiCad schematic)
At the start: 40 parts

Commit message: sketchingpad_proto1: routing done, no drc
Connections:
- no-connect marks 0 -> 1
Changed lines of the file:
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@@
 	(generator_version "10.0")
 	(paper "A4")
+	(no_connect
+		(at 121.92 143.51)
+	)
 	(wire
 		(pts

Commit message: extra input boost cap, stemmaqt/qwicc connector, added top decorative fill
Changed lines of the file:
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@@
 	(wire
 		(pts
-			(xy 20.32 43.18) (xy 34.29 43.18)
+			(xy 24.13 43.18) (xy 34.29 43.18)
 		)
 		(stroke
@@
 	)
 	(label "LED_DAT"
-		(at 20.32 43.18 0)
+		(at 24.13 43.18 0)
 		(effects
 			(font
@@
 		)
 	)
+	(global_label "LED_DAT"
+		(shape input)
+		(at 24.13 43.18 180)
+		(fields_autoplaced yes)
+		(effects
+			(font
+				(size 1.27 1.27)
+			)
+			(justify right)
+		)
+		(property "Intersheetrefs" "${INTERSHEET_REFS}"
+			(at 13.4039 43.18 0)
+			(hide yes)
+			(show_name no)
+			(do_not_autoplace no)
+			(effects
+				(font
+					(size 1.27 1.27)
+				)
+				(justify right)
+			)
+		)
+	)
