File: schematics/sketchingpad_stripproto1/sketchingpad_stripproto1.kicad_sch (KiCad schematic)
At the start: 75 parts, among them CN1 HC-1.0-4PWT, CN2 S2B-PH-SM4-TB, J1 Conn_01x07, J2 Conn_01x07, J3 Conn_01x03, Q1 AO3415A, SW1 TS-1088-AR02016, U1 TS20

Commit message: add arduino hwtest
Parts:
- renumbered C21 to C1, C26 to C10, C29 to C11, C32 to C12, C34 to C13, C36 to C14, C38 to C15, C40 to C16, C23 to C17, C24 to C18, C27 to C19, C25 to C2, C30 to C20, C28 to C3, C31 to C4, C33 to C5, C35 to C6, C37 to C7, C39 to C8, C22 to C9, LED21 to LED1, LED24 to LED10, LED29 to LED11, LED32 to LED12, LED34 to LED13, LED36 to LED14, LED38 to LED15, LED40 to LED16, LED23 to LED17, LED25 to LED18, LED27 to LED19, LED26 to LED2, LED30 to LED20, LED28 to LED3, LED31 to LED4, LED33 to LED5, LED35 to LED6, LED37 to LED7, LED39 to LED8, LED22 to LED9
Connections:
- net BUTTON: now also J1.3 (Pin_3); no longer J1.4 (Pin_4)
- net TS20_INT: now reaches R16.1, U1.19 (INT)
- net TS20_INT: now also J1.4 (Pin_4)
- no-connect marks 8 -> 7
