File: schematics/sketchingpad_stripproto1/sketchingpad_stripproto1.kicad_sch (KiCad schematic)
At the start: 75 parts, among them CN1 HC-1.0-4PWT, CN2 S2B-PH-SM4-TB, J1 Conn_01x07, J2 Conn_01x07, J3 Conn_01x03, Q1 AO3415A, SW1 TS-1088-AR02016, U1 TS20

Commit message: going with SMD-mounted XIAO I guess, added audio. ERC clean
Parts:
- removed J1, J2: Conn_01x07, easyeda2kicad:HDR-SMD_7P-P2.54_HX-PM2.54-1X7P-TP-YQ, symbol Connector_Generic:Conn_01x07
- removed J3: Conn_01x03, Connector_PinSocket_2.54mm:PinSocket_1x03_P2.54mm_Vertical, symbol PCM_4ms_Connector:Conn_01x03
- added C21: 100n, Capacitor_SMD:C_0603_1608Metric, symbol Device:C
- added C22: 47u, Capacitor_SMD:C_0603_1608Metric, symbol Device:C
- added J3: AudioJack4, todbot_stuff:Jack_3.5mm_PJ320D_Horizontal, symbol Connector_Audio:AudioJack4
- added R21: 220, Resistor_SMD:R_0603_1608Metric, symbol Device:R
- added R22: 100, Resistor_SMD:R_0603_1608Metric, symbol Device:R
- added R23: 1.8k, Resistor_SMD:R_0603_1608Metric, symbol Device:R
- added U2: Seeeduino Xiao nRF52840, PCM_marbastlib-xp-promicroish:Xiao_nRF52840_ACH, symbol PCM_marbastlib-promicroish:Seeeduino_Xiao_nRF52840
Connections:
- net +3.3V: now also U2.10 (3V3)
- net BUTTON: now also U2.3 (P0.28)
- net GND: now also C21.2, J3.R2, J3.S, R22.1, R23.1, U2.15 (BAT-), U2.9 (GND)
- net LED_POWER: now also U2.14 (P1.12)
- net PWM_AUDIO: now also R21.2, U2.1 (P0.02)
- net SCL: now also U2.6 (P0.05)
- net SDA: now also U2.5 (P0.04)
- net TS20_INT: now also U2.4 (P0.29)
- net VBAT: now also U2.16 (BAT+)
- net LED_DAT renamed LED_DATA
- net LED_DATA: now also U2.7 (P1.11)
- new net: C22.1, J3.R1, J3.T, R23.2
- new net: C21.1, C22.2, R21.1, R22.2
- no-connect marks 7 -> 12
Other:
- note added: "XIAO/QTPY"
- note removed: "HX PM2.54-1X7P TP-YQ"
- note removed: "XIAO / QTPY"
- moved on the sheet: CN1, CN2, Q1, R19, SW1

Commit message: final on the sketchingpad_stripproto1 sch maybe
Parts:
- added SW2: MINI MSK12CO2, easyeda2kicad:SW-SMD_MSK12CO2, symbol easyeda2kicad:MINIMSK12CO2
- added TP21, TP22: TestPoint, TestPoint:TestPoint_Pad_D1.5mm, symbol Connector:TestPoint
- U2: footprint PCM_marbastlib-xp-promicroish:Xiao_nRF52840_ACH -> todbot_stuff:Xiao_nRF52840_ACH-todedit
Connections:
- net GND: now also SW2.4, SW2.5, TP22.1
- net VBAT: now also SW2.2; no longer CN2.2
- new net: CN2.2, SW2.3, TP21.1
- no-connect marks 12 -> 13
Other:
- moved on the sheet: CN2, SW1

Commit message: more routed
Parts:
- removed SW1: TS-1088-AR02016, easyeda2kicad:SW-SMD_L3.9-W3.0-P4.45, symbol easyeda2kicad:TS-1088-AR02016
- removed U2: Seeeduino Xiao nRF52840, todbot_stuff:Xiao_nRF52840_ACH-todedit, symbol PCM_marbastlib-promicroish:Seeeduino_Xiao_nRF52840
- added SW1: TC-S3601-3.5-260G-F0.6, easyeda2kicad:SW-SMD_TC-S3601-3.5-260G-F0.6, symbol easyeda2kicad:TC-S3601-3.5-260G-F0.6
- added U2: Seeeduino Xiao nRF52840, todbot_stuff:Xiao_nRF52840_ACH-todedit, symbol todbot_stuff:Seeeduino_Xiao_nRF52840
- LED1, LED10, LED11, LED12, LED13, LED14, LED15, LED16, LED17, LED18, LED19, LED2, LED20, LED3, LED4, LED5, LED6, LED7, LED8, LED9: footprint easyeda2kicad:LED-SMD_4P-L4.0-W1.6-L -> todbot_stuff:LED-SMD_4P-L4.0-W1.6-L-todedits
- renumbered C100 to C23, R16 to R1, R18 to R2, R17 to R3, R19 to R4, R21 to R5, R22 to R6, R23 to R7
Connections:
- net +3.3V: now also U2.10 (3V3)
- net BUTTON: now also SW1.1, U2.11 (P1.15)
- net GND: now also SW1.2, SW1.3, SW1.4, U2.15 (BAT-), U2.9 (GND)
- net LED_DATA: now also U2.7 (P1.11)
- net LED_POWER: now also U2.14 (P1.12)
- net PWM_AUDIO: now also U2.1 (P0.02)
- net SCL: now also U2.6 (P0.05)
- net SDA: now also U2.5 (P0.04)
- net TOUCH1: now also U1.25 (CS1); no longer U1.17 (CS19)
- net TOUCH10: now also U1.16 (CS18); no longer U1.6 (CS9)
- net TOUCH11: now also U1.17 (CS19); no longer U1.16 (CS18)
- net TOUCH12: now also U1.18 (CS20); no longer U1.25 (CS1)
- net TOUCH13: now also U1.11 (CS13); no longer U1.8 (CS11)
- net TOUCH14: now also U1.12 (CS14); no longer U1.9 (CS12)
- net TOUCH15: now also U1.13 (CS15); no longer U1.15 (CS17)
- net TOUCH17: now also U1.1 (CS5); no longer U1.13 (CS15)
- net TOUCH18: now also U1.2 (CS6); no longer U1.12 (CS14)
- net TOUCH19: now also U1.3 (CS7); no longer U1.11 (CS13)
- net TOUCH3: now also U1.27 (CS3); no longer U1.28 (CS4)
- net TOUCH4: now also U1.28 (CS4); no longer U1.1 (CS5)
- net TOUCH5: now also U1.6 (CS9); no longer U1.3 (CS7)
- net TOUCH7: now also U1.8 (CS11); no longer U1.18 (CS20)
- net TOUCH8: now also U1.9 (CS12); no longer U1.27 (CS3)
- net TOUCH9: now also U1.15 (CS17); no longer U1.2 (CS6)
- net TS20_INT: now also U2.4 (P0.29)
- net VBAT: now also U2.16 (BAT+)

Commit message: more routed
Parts:
- added TP23: TestPoint, TestPoint:TestPoint_Pad_D1.5mm, symbol Connector:TestPoint
Connections:
- net 3V3_LED: now also TP23.1
Changed lines of the file:
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@@
 	)
 	(junction
+		(at 76.2 134.62)
+		(diameter 0)
+		(color 0 0 0 0)
+	)
+	(junction
 		(at 139.7 39.37)
 		(diameter 0)
@@
 					(unit 1)
 				)
+			)
+		)
+	)
+	(symbol
+		(lib_id "Connector:TestPoint")
+		(at 76.2 134.62 270)
+		(unit 1)
+		(body_style 1)
+		(exclude_from_sim no)
+		(in_bom yes)
+		(on_board yes)
+		(in_pos_files yes)
+		(dnp no)
+		(fields_autoplaced yes)
+		(property "Reference" "TP23"
+			(at 81.28 133.3499 90)
+			(show_name no)
+			(do_not_autoplace no)
+			(effects
+				(font
+					(size 1.27 1.27)
+				)
+				(justify left)
+			)
+		)
+		(property "Value" "TestPoint"
+			(at 81.28 135.8899 90)
+			(show_name no)
+			(do_not_autoplace no)
+			(effects
+				(font
+					(size 1.27 1.27)
+				)
+				(justify left)
+			)
+		)
+		(property "Footprint" "TestPoint:TestPoint_Pad_D1.5mm"
+			(at 76.2 139.7 0)
+			(hide yes)
+			(show_name no)
+			(do_not_autoplace no)
+			(effects
+				(font
+					(size 1.27 1.27)
+				)
+			)
+		)
+		(property "Datasheet" ""
+			(at 76.2 139.7 0)
+			(hide yes)
+			(show_name no)
+			(do_not_autoplace no)
+			(effects
+				(font
+					(size 1.27 1.27)
+				)
+			)
+		)
+		(property "Description" "test point"
+			(at 76.2 134.62 0)
+			(hide yes)
+			(show_name no)
+			(do_not_autoplace no)
+			(effects
+				(font
+					(size 1.27 1.27)
+				)
+			)
+		)
+		(property "LCSC Part" ""
+			(at 76.2 134.62 0)
+			(hide yes)
+			(show_name no)
+			(do_not_autoplace no)
+			(effects
+				(font
+					(size 1.27 1.27)
+				)
+			)
+		)
+		(property "DigikeyPN" ""
+			(at 76.2 134.62 0)
+			(hide yes)
+			(show_name no)
+			(do_not_autoplace no)
+			(effects
+				(font
+					(size 1.27 1.27)
+				)
+			)
+		)
+		(property "MPN" ""
+			(at 76.2 134.62 0)
+			(hide yes)
+			(show_name no)
+			(do_not_autoplace no)
+			(effects
+				(font
+					(size 1.27 1.27)
+				)
+			)
+		)
+		(property "Note" ""
+			(at 76.2 134.62 0)
+			(show_name no)
+			(do_not_autoplace no)
+			(effects
+				(font
+					(size 1.27 1.27)
+				)
+			)
+		)
+		(pin "1"
+		)
+		(instances
+			(project "sketchingpad_stripproto1"
+				(path "/69aff514-3aa6-493d-bc6d-4103dc0ce10d"
+					(reference "TP23")
+					(unit 1)
+				)

Commit message: ERC and DRC pass
Parts:
- TP23: value TestPoint -> 3V3_LED
- renumbered J3 to J1
Changed lines of the file:
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@@
 	(paper "A3")
 	(rectangle
-		(start 47.879 22.479)
-		(end 68.834 42.799)
+		(start 48.26 22.479)
+		(end 68.58 42.799)
 		(stroke
 			(width 0)
@@
 	(text "A0/D0\nA1/D1\nA2/D2\nA3/D3\nSDA/D4\nSCL/D5\nTX/D6"
 		(exclude_from_sim no)
-		(at 48.26 33.02 0)
+		(at 48.768 33.02 0)
 		(effects
 			(font
@@
 	(text "5V\nGnd\n3V3\nMOSI\nMISO\nSCK\nRX"
 		(exclude_from_sim no)
-		(at 68.58 33.02 0)
+		(at 68.072 33.02 0)
 		(effects
 			(font
@@
 		(dnp no)
 		(fields_autoplaced yes)
-		(property "Reference" "J3"
+		(property "Reference" "J1"
 			(at 208.28 89.5349 0)
 			(show_name no)
@@
 			)
 		)
+		(property "DigikeyPN" ""
+			(at 199.39 92.71 0)
+			(hide yes)
+			(show_name no)
+			(do_not_autoplace no)
+			(effects
+				(font
+					(size 1.27 1.27)
+				)
+			)
+		)
+		(property "MPN" ""
+			(at 199.39 92.71 0)
+			(hide yes)
+			(show_name no)
+			(do_not_autoplace no)
+			(effects
+				(font
+					(size 1.27 1.27)
+				)
+			)
+		)
+		(property "Note" ""
+			(at 199.39 92.71 0)
+			(show_name no)
+			(do_not_autoplace no)
+			(effects
+				(font
+					(size 1.27 1.27)
+				)
+			)
+		)
 		(pin "S"
 		)
@@
 			(project "sketchingpad_stripproto1"
 				(path "/69aff514-3aa6-493d-bc6d-4103dc0ce10d"
-					(reference "J3")
+					(reference "J1")
 					(unit 1)
 				)
@@
 			)
 		)
-		(property "Value" "TestPoint"
+		(property "Value" "3V3_LED"
 			(at 81.28 135.8899 90)
 			(show_name no)
@@
 		(in_pos_files yes)
 		(dnp no)
-		(fields_autoplaced yes)
 		(property "Reference" "Q1"
-			(at 60.96 128.27 90)
+			(at 60.96 127.254 90)
 			(show_name no)
 			(do_not_autoplace no)
@@
 		)
 		(property "Value" "AO3415A"
-			(at 60.96 130.81 90)
+			(at 60.96 129.794 90)
 			(show_name no)
 			(do_not_autoplace no)
@@
 			(show_name no)
 			(do_not_autoplace no)
+			(effects
+				(font
+					(size 1.27 1.27)
+				)
+			)
+		)
+		(property "DigikeyPN" ""
+			(at 133.35 38.1 0)
+			(hide yes)
+			(show_name no)
+			(do_not_autoplace no)
+			(effects
+				(font
+					(size 1.27 1.27)
+				)
+			)
+		)
+		(property "Note" ""
+			(at 133.35 38.1 0)
+			(show_name no)
+			(do_not_autoplace no)
