File: schematics/sketchingpad1_mpr/sketchingpad1_mpr.kicad_pcb (KiCad board)
At the start: 4 copper layers, 158.5 x 66 mm, 85 parts, among them CN1 HC-1.0-4PWT, CN2 S2B-PH-SM4-TB, J1 AudioJack4, Q1 AO3415A, SW1 TC-S3601-3.5-260G-F0.6, SW2 MINI MSK12CO2, U2 Seeeduino Xiao nRF52840, U3 MPR121QR2, U4 MPR121QR2

Commit message: routed.  crap, TS20 out of stock at LCSC. respin with 2xMPR121
Parts:
- added C24: 100n, Capacitor_SMD:C_0603_1608Metric, B.Cu at (132.7, 113.4)
- added C25: 100n, Capacitor_SMD:C_0603_1608Metric, B.Cu at (138.0, 102.6)
- added C26: 100n, Capacitor_SMD:C_0603_1608Metric, B.Cu at (137.8, 112.7)
- added J2: Conn_01x04, Connector_PinHeader_1.27mm:PinHeader_2x02_P1.27mm_Vertical, F.Cu at (135.4, 122.8)
- added R8: 75, Resistor_SMD:R_0603_1608Metric, B.Cu at (140.0, 102.6)
- added R9: 75, Resistor_SMD:R_0603_1608Metric, B.Cu at (139.8, 112.7)
- moved C23 2.60 mm to (133.4, 101.8), turned to 90 degrees
Connections:
- U3 pad 4: unconnected-(U3-ADDR-Pad4) -> GND
- U3 pad 5: unconnected-(U3-VREG-Pad5) -> Net-(U3-VREG)
- U3 pad 7: unconnected-(U3-REXT-Pad7) -> Net-(U3-REXT)
- U4 pad 10: unconnected-(U4-ELE2-Pad10) -> /TOUCH15
- U4 pad 11: unconnected-(U4-ELE3-Pad11) -> /TOUCH16
- U4 pad 12: unconnected-(U4-ELE4-Pad12) -> /TOUCH24
- U4 pad 13: unconnected-(U4-ELE5-Pad13) -> /TOUCH22
- U4 pad 14: unconnected-(U4-ELE6-Pad14) -> /TOUCH21
- U4 pad 15: unconnected-(U4-ELE7-Pad15) -> /TOUCH23
- U4 pad 16: unconnected-(U4-ELE8-Pad16) -> /TOUCH9
- U4 pad 17: unconnected-(U4-ELE9-Pad17) -> /TOUCH10
- U4 pad 18: unconnected-(U4-ELE10-Pad18) -> /TOUCH11
- U4 pad 19: unconnected-(U4-ELE11-Pad19) -> /TOUCH12
- U4 pad 4: unconnected-(U4-ADDR-Pad4) -> +3.3V
- U4 pad 5: unconnected-(U4-VREG-Pad5) -> Net-(U4-VREG)
- U4 pad 7: unconnected-(U4-REXT-Pad7) -> Net-(U4-REXT)
- U4 pad 8: unconnected-(U4-ELE0-Pad8) -> /TOUCH13
- U4 pad 9: unconnected-(U4-ELE1-Pad9) -> /TOUCH14
Routing:
- net +3.3V: track 65.2 -> 82.4 mm, vias 4 -> 7
- net /SCL: track 46.5 -> 55.0 mm, vias 3 -> 4
- net /TOUCH_INT: track 49.3 -> 56.1 mm
- net /TOUCH23: track 0.00 -> 6.72 mm
- net /TOUCH24: track 0.00 -> 6.46 mm
- net Net-(U4-REXT): track 0.00 -> 5.13 mm
- net /TOUCH22: track 0.00 -> 4.64 mm
- net /TOUCH21: track 0.00 -> 4.47 mm
- net Net-(U3-REXT): track 0.00 -> 4.45 mm
- net GND: track 16.9 -> 20.7 mm
- net Net-(U4-VREG): track 0.00 -> 2.63 mm
- net Net-(U3-VREG): track 0.00 -> 2.45 mm
- net /TOUCH4: track 17.3 -> 15.7 mm
- net /SDA: track 50.0 -> 51.2 mm, vias 3 -> 4
- net /TOUCH10: track 51.1 -> 52.1 mm
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
Commit message: sketchingpad1_mpr: small header for unused touch pins
Parts:
- J2: moved to B.Cu
- R8, R9: value 75 -> 75k
- moved J2 1.11 mm to (135.4, 123.9)
Connections:
- J2 pad 1: /TOUCH21 -> /TOUCH23
- J2 pad 2: /TOUCH22 -> /TOUCH24
- J2 pad 3: /TOUCH23 -> /TOUCH21
- J2 pad 4: /TOUCH24 -> /TOUCH22
Routing:
- net /TOUCH12: track 17.4 -> 14.4 mm
- net /TOUCH13: track 16.9 -> 14.2 mm
- net /TOUCH14: track 34.4 -> 33.9 mm
Other:
- board text added: "21 23"
- board text added: "22 24"
- board text added: "sketchingpad1_mpr 17 Sep 2026 @todbot"
- board text removed: "sketchingpad1 17 Sep 2026 @todbot"
