File: schematics/sketchingpad1_mpr/sketchingpad1_mpr.kicad_sch (KiCad schematic)
At the start: 84 parts, among them CN1 HC-1.0-4PWT, CN2 S2B-PH-SM4-TB, J1 AudioJack4, Q1 AO3415A, SW1 TC-S3601-3.5-260G-F0.6, SW2 MINI MSK12CO2, U2 Seeeduino Xiao nRF52840, U3 MPR121QR2, U4 MPR121QR2

Commit message: routed.  crap, TS20 out of stock at LCSC. respin with 2xMPR121
Parts:
- added C24, C25, C26: 100n, Capacitor_SMD:C_0603_1608Metric, symbol Device:C
- added J2: Conn_01x04, Connector_PinHeader_1.27mm:PinHeader_2x02_P1.27mm_Vertical, symbol Connector_Generic:Conn_01x04
- added R8, R9: 75, Resistor_SMD:R_0603_1608Metric, symbol Device:R
Connections:
- net +3.3V: now also U4.4 (ADDR), C24.1
- net GND: now also U3.4 (ADDR), C24.2, C25.2, C26.2, R8.2, R9.2
- net TOUCH1: now also U3.14 (ELE6)
- net TOUCH10: now also U4.17 (ELE9)
- net TOUCH11: now also U4.18 (ELE10)
- net TOUCH12: now also U4.19 (ELE11)
- net TOUCH13: now also U4.8 (ELE0)
- net TOUCH14: now also U4.9 (ELE1)
- net TOUCH15: now also U4.10 (ELE2)
- net TOUCH16: now also U4.11 (ELE3)
- net TOUCH17: now also U3.18 (ELE10)
- net TOUCH18: now also U3.19 (ELE11)
- net TOUCH19: now also U3.8 (ELE0)
- net TOUCH2: now also U3.15 (ELE7)
- net TOUCH20: now also U3.9 (ELE1)
- net TOUCH3: now also U3.16 (ELE8)
- net TOUCH4: now also U3.17 (ELE9)
- net TOUCH5: now also U3.10 (ELE2)
- net TOUCH6: now also U3.11 (ELE3)
- net TOUCH7: now also U3.12 (ELE4)
- net TOUCH8: now also U3.13 (ELE5)
- net TOUCH9: now also U4.16 (ELE8)
- net at U3.5 (VREG): now also C25.1
- net at U3.7 (REXT): now also R8.1
- net TOUCH24: now reaches U4.12 (ELE4)
- net TOUCH24: now also J2.4 (Pin_4)
- net TOUCH22: now reaches U4.13 (ELE5)
- net TOUCH22: now also J2.2 (Pin_2)
- net TOUCH21: now reaches U4.14 (ELE6)
- net TOUCH21: now also J2.1 (Pin_1)
- net TOUCH23: now reaches U4.15 (ELE7)
- net TOUCH23: now also J2.3 (Pin_3)
- net at U4.5 (VREG): now also C26.1
- net at U4.7 (REXT): now also R9.1
Other:
- moved on the sheet: C23

Commit message: fix 75->75k mpr resistors. routed.  crap, TS20 out of stock at LCSC. respin with 2xMPR121
Parts:
- R8, R9: value 75 -> 75k
Changed lines of the file:
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@@
 			)
 		)
-		(property "Value" "75"
+		(property "Value" "75k"
 			(at 233.172 106.426 90)
 			(show_name no)
@@
 			)
 		)
-		(property "Value" "75"
+		(property "Value" "75k"
 			(at 235.712 154.686 90)
 			(show_name no)

Commit message: sketchingpad1_mpr: small header for unused touch pins
Parts:
- J2: now left out of the parts list
Connections:
- net TOUCH21: now also J2.3 (Pin_3); no longer J2.1 (Pin_1)
- net TOUCH22: now also J2.4 (Pin_4); no longer J2.2 (Pin_2)
- net TOUCH23: now also J2.1 (Pin_1); no longer J2.3 (Pin_3)
- net TOUCH24: now also J2.2 (Pin_2); no longer J2.4 (Pin_4)
Changed lines of the file:
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@@
 		)
 	)
-	(label "TOUCH22"
+	(label "TOUCH24"
 		(at 262.89 177.8 0)
 		(effects
@@
 		)
 	)
-	(label "TOUCH21"
+	(label "TOUCH23"
 		(at 262.89 175.26 0)
 		(effects
@@
 		)
 	)
-	(label "TOUCH23"
+	(label "TOUCH21"
 		(at 262.89 180.34 0)
 		(effects
@@
 		)
 	)
-	(label "TOUCH24"
+	(label "TOUCH22"
 		(at 262.89 182.88 0)
 		(effects
@@
 		(body_style 1)
 		(exclude_from_sim no)
-		(in_bom yes)
+		(in_bom no)
 		(on_board yes)
-		(in_pos_files yes)
+		(in_pos_files no)
 		(dnp no)
 		(fields_autoplaced yes)
